File: TOBI.kicad_sch (KiCad schematic)
At the start: 23 parts, among them J1 Battery Connector, J2 Top Screw Terminal, J3 Bottom Screw Terminal, Q1 Q_NMOS_GDS, Q2 Q_NMOS_GDS, Q3 Q_NMOS_GDS, U1 XIAO-ESP32-S3-SMD, U2 LSM6DSO32, U4 MS5611-01BA

Commit message: Final Schematics
Checked schematics and parts
Parts:
- R1, R10, R11, R2, R3, R4, R5, R6, R7, R8, R9: footprint (none) -> Resistor_SMD:R_01005_0402Metric
Connections:
- net +3.3V: no longer U2.11 (SCL)
- net -BATT: no longer C3.1, C4.1, C5.1, Q1.3 (S), Q2.3 (S), Q3.3 (S), R1.1, R3.1, R4.1, R6.1, R7.1, R9.1, U1.13 (GND), U2.3 (CS), U2.4 (SDX), U2.5 (SCX), U4.3 (GND), U4.4 (CSB), U4.5 (CSB)
- net APPO: now also Q1.2 (D), R2.1
- net MAIN: now also Q2.2 (D), R5.1
- net MOTOR: now also Q3.2 (D), R8.1
- net SCL: now also R10.2, U1.6 (GPIO6_A5_D5_SCL), U2.11 (SCL)
- net SDA: now also R11.2, U1.5 (GPIO5_A4_D4_SDA), U2.10 (SDA)
- net CONT 2: now reaches R5.2, R6.2
- net CONT 2: now also U1.11 (GPIO9_A10_D10_MOSI)
- net IGNIT 2: now reaches Q2.1 (G), R4.2
- net IGNIT 2: now also U1.10 (GPIO8_A9_D9_MISO)
- net GND: now reaches U2.12 (GND)
- net GND: now also C3.1, C4.1, C5.1, Q1.3 (S), Q2.3 (S), Q3.3 (S), R1.1, R3.1, R4.1, R6.1, R7.1, R9.1, U1.13 (GND), U2.3 (CS), U2.4 (SDX), U2.5 (SCX), U4.3 (GND), U4.4 (CSB), U4.5 (CSB)
- net CONT 3: now reaches R8.2, R9.2
- net CONT 3: now also U1.1 (GPIO1_A0_D0)
- net IGNIT 1: now reaches Q1.1 (G), R3.2
- net IGNIT 1: now also U1.4 (GPIO4_A3_D3)
- net CONT 1: now reaches R1.2, R2.2
- net CONT 1: now also U1.3 (GPIO3_A2_D2)
- net IGNIT 3: now reaches Q3.1 (G), R7.2
- net IGNIT 3: now also U1.2 (GPIO2_A1_D1)
- no-connect marks 19 -> 21
Other:
- note added: "-BATT INSTEAD OF GND"
- note removed: "APPO"
- note removed: "CONT 1"
- note removed: "CONT 2"
- note removed: "CONT 3"
- note removed: "IGNIT 1"
- note removed: "IGNIT 2"
- note removed: "IGNIT 3"
- note removed: "MAIN"
- note removed: "MOTOR"
- note removed: "SCL"
- note removed: "SDA"
- moved on the sheet: C3, C4, J2, J3, U2

Commit message: Modified ESP32S3 Footprint
Incorrect footprint for the ESP, updated and modified the PCB for re-wiring.
Parts:
- U1: footprint Library:ESP32S3 -> Seeed_Studio_XIAO_Series:XIAO-ESP32-S3-DIP
Changed lines of the file:
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@@
 			)
 		)
-		(property "Footprint" "Library:ESP32S3"
+		(property "Footprint" "Seeed_Studio_XIAO_Series:XIAO-ESP32-S3-DIP"
 			(at 125.73 38.1 0)
 			(effects

Commit message: Final PCB
Final PCB that is being pushed out, DRC checks fine
Connections:
- net GND is gone; now on net -BATT: C3.1, C4.1, C5.1, Q1.3 (S), Q2.3 (S), Q3.3 (S), R1.1, R3.1, R4.1, R6.1, R7.1, R9.1, U1.13 (GND), U2.12 (GND), U2.3 (CS), U2.4 (SDX), U2.5 (SCX), U4.3 (GND), U4.4 (CSB), U4.5 (CSB)
Changed lines of the file:
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@@
 		(on_board yes)
 		(dnp no)
-		(fields_autoplaced yes)
 		(property "Reference" "#PWR022"
 			(at 194.31 30.48 0)
@@
 			)
 		)
-		(property "Value" "GND"
-			(at 194.31 21.59 0)
+		(property "Value" "-BATT"
+			(at 191.008 22.352 0)
 			(effects
 				(font
 					(size 1.27 1.27)
 				)
+				(justify left)
 			)
 		)
